File: preliminary block diagram/rev1_block_diagram.kicad_sch (KiCad schematic)
At the start: 15 parts, among them SW1 ???, U29 LMX2594+100MHz oscillator, U30 ????, U31 HMC451?, U32 ????, U33 ADP-2-1W, U35 Mixer, U37 Mixer, U39 ADP-2-1W

Commit message: udated diagram
Parts:
- FL1, FL2: value LP???? -> LP
- FL3, FL4: value BP 10-12GHz???? -> BP 10-12GHz
- U30: value ???? -> PA
- U31: value HMC451? -> HMC451
- U32: value ???? -> LNA
Changed lines of the file:
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@@
 		(on_board yes)
 		(dnp no)
-		(fields_autoplaced yes)
 		(property "Reference" "SW1"
-			(at 198.12 81.28 0)
+			(at 198.374 83.82 0)
 			(effects
 				(font
@@
 					(size 1.27 1.27)
 				)
+				(hide yes)
 			)
 		)
@@
 			)
 		)
-		(property "Value" "????"
+		(property "Value" "LNA"
 			(at 220.218 102.108 0)
 			(effects
@@
 			)
 		)
-		(property "Value" "BP 10-12GHz????"
+		(property "Value" "BP 10-12GHz"
 			(at 220.98 72.39 0)
 			(effects
@@
 			)
 		)
-		(property "Value" "????"
+		(property "Value" "PA"
 			(at 242.57 76.2 0)
 			(effects
@@
 			)
 		)
-		(property "Value" "HMC451?"
+		(property "Value" "HMC451"
 			(at 92.71 83.82 0)
 			(effects
@@
 			)
 		)
-		(property "Value" "LP????"
-			(at 170.18 129.032 90)
+		(property "Value" "LP"
+			(at 166.37 129.032 90)
 			(effects
 				(font
@@
 		(on_board yes)
 		(dnp no)
-		(fields_autoplaced yes)
 		(property "Reference" "FL1"
-			(at 129.54 126.9999 90)
-			(effects
-				(font
-					(size 1.27 1.27)
-				)
-				(justify left)
-			)
-		)
-		(property "Value" "LP????"
-			(at 129.54 129.5399 90)
-			(effects
-				(font
-					(size 1.27 1.27)
-				)
-				(justify left)
+			(at 124.968 127.254 90)
+			(effects
+				(font
+					(size 1.27 1.27)
+				)
+				(justify right)
+			)
+		)
+		(property "Value" "LP"
+			(at 125.73 129.794 90)
+			(effects
+				(font
+					(size 1.27 1.27)
+				)
+				(justify right)
 			)
 		)
@@
 			)
 		)
-		(property "Value" "BP 10-12GHz????"
+		(property "Value" "BP 10-12GHz"
 			(at 243.84 95.25 0)
 			(effects
